File: pcf8583-tester/RTC Tester.kicad_sch (KiCad schematic)
At the start: 8 parts, among them IC1 PCF8583P_F5,112

Commit message: Title blocks: copyright Arley Silveira, credit to Alvaro Alea Fernandez, licence
Other:
- company: (none) -> Arley Silveira
- title: (none) -> PCF8583 Tester
Changed lines of the file:
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@@
 	(generator_version "10.0")
 	(paper "A4")
+	(title_block
+		(title "PCF8583 Tester")
+		(company "Arley Silveira")
+		(comment 1 "Copyright (c) 2026 Arley Silveira")
+		(comment 2 "Licence: CERN-OHL-S v2")
+	)
 	(junction
 		(at 81.534 82.55)
