File: QL_Minerva_MK2.kicad_pcb (KiCad board)
At the start: 2 copper layers, 42.7 x 40.6 mm, 19 parts, among them J1 Conn_01x02_Pin, J2 Conn_01x05_Pin, SW1 SW_SPDT, U1 Socket to QL, U3 PCF8583P, U4 GAL16V8, U5 74LS133, U6 27C512PLCC, Y1 32.768 kHz

Commit message: Add C5 10uF bulk capacitor on +5V
Parts:
- added C5: 10uf, Capacitor_SMD:C_0805_2012Metric, B.Cu at (94.9, 65.0)
Routing:
- net +5V: track 107.8 -> 112.9 mm, vias 10 -> 11
