File: QL_Minerva_MK2.kicad_sch (KiCad schematic)
At the start: 18 parts, among them J1 Conn_01x02_Pin, J2 Conn_01x05_Pin, SW1 SW_SPDT, U1 Socket to QL, U3 PCF8583P, U4 GAL16V8, U5 74LS133, U6 27C512PLCC, Y1 32.768 kHz

Commit message: Title blocks: copyright Arley Silveira, credit to Alvaro Alea Fernandez, licence
Other:
- company: Alvaro Alea Fernandez -> Arley Silveira
Changed lines of the file:
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@@
 		(date "2025-04-08")
 		(rev "0.2")
-		(company "Alvaro Alea Fernandez")
+		(company "Arley Silveira")
+		(comment 1 "Copyright (c) 2026 Arley Silveira - SMD redesign")
+		(comment 2 "Based on the KiCad capture (c) 2024 Alvaro Alea Fernandez")
+		(comment 3 "Licence: CERN-OHL-S v2")
 	)
 	(text_box "NOTE:\n\nOn QL's PCB pins 1 and 28 of ROM's Slot are interconected to +5V. So once conected to the QL the Vcc and +5V are the same potential, has been diferenciate in the schematic with the only propouse to match the original PCB."

Commit message: Add C5 10uF bulk capacitor on +5V
Parts:
- added C5: 10uf, Capacitor_SMD:C_0805_2012Metric, symbol Other:C_Small
Connections:
- net +5V: now also C5.1
- net GND: now also C5.2
